File: Infra-pHAT.sch (KiCad schematic (older format))
At the start: 0 parts

Commit message: populated the schematic
Parts:
- added C1: 0.1, Capacitors_SMD:C_0603_HandSoldering, symbol C
- added C2: 4.7, Capacitors_SMD:C_0805_HandSoldering, symbol CP
- added IRRX1: TSOP34838, myfootprint:TSOP38X, symbol TSOP382
- added IRTX1, IRTX2: L-53F3BT, LEDs:LED-5MM, symbol LED
- added JP1: JUMPER, Pin_Headers:Pin_Header_Straight_1x02, symbol JUMPER
- added Q1: BC817, TO_SOT_Packages_SMD:SOT-23, symbol Q_NPN_BEC
- added R1: 1K, Resistors_SMD:R_0603_HandSoldering, symbol R
- added R2, R3, R6, R7: 4.7K, Resistors_SMD:R_0603_HandSoldering, symbol R
- added R4: 10K, Resistors_SMD:R_0603_HandSoldering, symbol R
- added R5: 470, Resistors_SMD:R_0603_HandSoldering, symbol R
- added RASP_CONN1: Raspberry_PI, Pin_Headers:Pin_Header_Straight_2x20, symbol Raspberry_PI
- added SENS1, SENS2, SENS3: I2C_SENS_1, Pin_Headers:Pin_Header_Straight_1x04, symbol I2C_SENS_1
- added U1: CAT24C32WI-GT3, Housings_DIP:DIP-8_W7.62mm, symbol CAT24C32WI-GT3
- added UART1: CONN_01X04, Pin_Headers:Pin_Header_Straight_1x04, symbol CONN_01X04
Connections:
- new net: IRTX1.1 (K), Q1.3 (C)
- new net: IRTX1.2 (A), IRTX2.1 (K)
- new net +3V3: RASP_CONN1.1 (VDD(3.3V))
- new net +5V: RASP_CONN1.2 (VPP(5V))
- new net GND: C1.2, C2.2, IRRX1.2 (GND), JP1.2
- no-connect marks 0 -> 20

Commit message: Schematic Complete.
Connections:
- net +3V3: now also C1.1, R1.1, R2.1, R3.1, R5.1, R6.1, R7.1, RASP_CONN1.17 (VDD(3.3V)), SENS1.1 (VIN), SENS2.1 (VIN), SENS3.1 (VIN), U1.8 (VCC), UART1.1 (P1)
- net +5V: now also IRTX2.2 (A), RASP_CONN1.4 (Vpp(5V))
- net GND: now also Q1.2 (E), R4.1, RASP_CONN1.14 (GND), RASP_CONN1.20 (GND), RASP_CONN1.25 (GND), RASP_CONN1.30 (GND), RASP_CONN1.34 (GND), RASP_CONN1.39 (GND), RASP_CONN1.6 (GND), RASP_CONN1.9 (GND), SENS1.2 (GND), SENS2.2 (GND), SENS3.2 (GND), U1.1 (A0), U1.2 (A1), U1.3 (A2), U1.4 (VSS), UART1.4 (P4)
- net RXD: now also RASP_CONN1.10 (GPIO15/UART_RXD), UART1.3 (P3)
- net TXD: now also RASP_CONN1.8 (GPIO14/UART_TXD), UART1.2 (P2)
- net at U1.5 (SDA): now also R3.2, RASP_CONN1.27 (ID_SD)
- net at U1.6 (SCL): now also R2.2, RASP_CONN1.28 (ID_SC)
- net at U1.7 (WP): now also JP1.1, R1.2
- net at RASP_CONN1.11 (GPIO17): now also Q1.1 (B), R4.2
- net at RASP_CONN1.12 (GPIO18/PCM_CLK): now also IRRX1.1 (Out)
- net at RASP_CONN1.3 (GPIO2/I2C1_SDA): now also R6.2, SENS1.4 (SDA), SENS2.4 (SDA), SENS3.4 (SDA)
- net at RASP_CONN1.5 (GPIO3/I2C1_SCL): now also R7.2, SENS1.3 (SCL), SENS2.3 (SCL), SENS3.3 (SCL)
- net at IRRX1.3 (Vss): now also C2.1, R5.2
Changed lines of the file:
@@
 NoConn ~ 5350 2600
 NoConn ~ 5350 2700
+Wire Wire Line
+	950  3500 800  3500
+Wire Wire Line
+	800  3500 800  3950
+Wire Wire Line
+	950  3600 800  3600
+Connection ~ 800  3600
+Wire Wire Line
+	950  3700 800  3700
+Connection ~ 800  3700
+Wire Wire Line
+	950  3800 800  3800
+Connection ~ 800  3800
+Wire Wire Line
+	2200 3500 2050 3500
+Connection ~ 2200 3050
+Wire Wire Line
+	2950 3050 2950 3200
+Wire Wire Line
+	2800 3050 2800 3200
+Connection ~ 2800 3050
+Wire Wire Line
+	2650 3200 2650 3050
+Connection ~ 2650 3050
+Wire Wire Line
+	2200 3050 2950 3050
+Wire Wire Line
+	2050 3600 2650 3600
+Wire Wire Line
+	2650 3500 2650 4050
+Wire Wire Line
+	2800 3700 2800 3500
+Wire Wire Line
+	2950 3800 2950 3500
+Connection ~ 2950 3800
+Connection ~ 2800 3700
+Wire Wire Line
+	2200 2700 2200 3500
+Connection ~ 2650 3600
+Wire Wire Line
+	7500 4750 7500 5300
+Connection ~ 7500 5150
+Wire Wire Line
+	3450 2150 3450 2250
+Connection ~ 3450 2150
+Connection ~ 3450 1800
+Wire Wire Line
+	3450 1800 3450 1900
+Wire Wire Line
+	5350 1800 7000 1800
+Wire Wire Line
+	5350 1900 7000 1900
+Connection ~ 6650 1800
+Connection ~ 6800 1900
+Wire Wire Line
+	8050 900  8050 2100
+Wire Wire Line
+	8050 1900 7900 1900
+Connection ~ 7900 1800
+Wire Wire Line
+	2050 3700 3450 3700
+Wire Wire Line
+	2050 3800 3450 3800
+Wire Wire Line
+	7850 5150 7900 5150
+Wire Wire Line
+	7550 5150 7500 5150
+Wire Wire Line
+	5350 4150 5850 4150
+Wire Wire Line
+	5850 4150 5850 4850
+Wire Wire Line
+	5850 4850 7400 4850
+Wire Wire Line
+	7400 4850 7400 4750
+Wire Wire Line
+	6500 2450 6500 2600
+Wire Wire Line
+	8800 2400 8550 2400
+Wire Wire Line
+	8550 2100 8800 2100
+Wire Wire Line
+	5350 2200 5500 2200
+Wire Wire Line
+	5350 2300 5500 2300
+Wire Wire Line
+	8800 2200 8550 2200
+Wire Wire Line
+	8800 2300 8550 2300
+Connection ~ 7900 1200
+Connection ~ 7900 800
+Wire Wire Line
+	7900 900  8050 900
+Wire Wire Line
+	8050 1300 7900 1300
+Connection ~ 8050 1900
+Connection ~ 8050 1300
+Wire Wire Line
+	7000 800  6650 800
+Wire Wire Line
+	6200 1200 7000 1200
+Connection ~ 6650 1200
+Wire Wire Line
+	7000 900  6800 900
+Wire Wire Line
+	6350 1300 7000 1300
+Connection ~ 6800 1300
+Wire Wire Line
+	6350 1050 6350 1300
+Wire Wire Line
+	6200 1050 6200 1200
+Wire Wire Line
+	6050 750  6350 750
+Connection ~ 6200 750
+Wire Wire Line
+	5850 4050 5350 4050
+Wire Wire Line
+	6800 900  6800 1900
+Wire Wire Line
+	6650 800  6650 1800
+Wire Wire Line
+	7900 700  7900 1800
+Wire Wire Line
+	5850 4050 5850 3600
+Wire Wire Line
+	5850 3600 6200 3600
+Wire Wire Line
+	6200 3600 6200 3750
+Wire Wire Line
+	6200 4050 6200 4250
+Wire Wire Line
+	6500 3800 6500 4250
+Wire Wire Line
+	3450 2650 3450 3450
 Connection ~ 3450 2750
 Connection ~ 3450 2850
